File: KiCAD/Joule-Thief.kicad_pcb (KiCad board)
At the start: 2 copper layers, 0 parts

Commit message: new pcb revision
Parts:
- added BATT_1: Alkaline AA, Joule Thief-Library:AA_Cell_Clip, F.Cu at (130.8, 92.7)
- added BT1: Battery_Cell, Joule Thief-Library:18650_Cell_Clip, F.Cu at (140.3, 71.6)
- added C1: 0.1u, Capacitor_SMD:C_0805_2012Metric_Pad1.18x1.45mm_HandSolder, F.Cu at (142.0, 108.9)
- added C10: 0.1u, Capacitor_SMD:C_0805_2012Metric_Pad1.18x1.45mm_HandSolder, F.Cu at (182.0, 86.6)
- added C2: 0.1u, Capacitor_SMD:C_0805_2012Metric_Pad1.18x1.45mm_HandSolder, F.Cu at (148.7, 104.7)
- added C3: 100u, Capacitor_SMD:C_0805_2012Metric_Pad1.18x1.45mm_HandSolder, F.Cu at (157.6, 104.2)
- added C4: 10u, Capacitor_SMD:C_0805_2012Metric_Pad1.18x1.45mm_HandSolder, F.Cu at (163.4, 99.1)
- added C5: 1u, Capacitor_SMD:C_0805_2012Metric_Pad1.18x1.45mm_HandSolder, F.Cu at (160.8, 107.4)
- added C6: 0.1u, Capacitor_SMD:C_0805_2012Metric_Pad1.18x1.45mm_HandSolder, F.Cu at (171.3, 104.8)
- added C7: 4.7u, Capacitor_SMD:C_0805_2012Metric_Pad1.18x1.45mm_HandSolder, F.Cu at (168.7, 104.8)
- added C8: 0.1u, Capacitor_SMD:C_0805_2012Metric_Pad1.18x1.45mm_HandSolder, F.Cu at (118.7, 109.3)
- added C9: 0.1u, Capacitor_SMD:C_0805_2012Metric_Pad1.18x1.45mm_HandSolder, F.Cu at (126.2, 104.9)
- added J2: Conn_01x06_Socket, Connector_PinSocket_2.54mm:PinSocket_1x06_P2.54mm_Vertical, F.Cu at (166.0, 111.3)
- added L1: 10u, Joule Thief-Library:Power_Inductor_101040, F.Cu at (167.6, 90.6)
- added Q1: AO3400A, Package_TO_SOT_SMD:SOT-23, F.Cu at (182.2, 97.0)
- added Q2: AO3400A, Package_TO_SOT_SMD:SOT-23, F.Cu at (177.1, 90.5)
- added R1: 10, Resistor_SMD:R_0805_2012Metric_Pad1.20x1.40mm_HandSolder, F.Cu at (144.7, 102.9)
- added R10: 0.1R, Resistor_SMD:R_Shunt_Vishay_WSK2512_6332Metric_T1.19mm, F.Cu at (130.6, 107.3)
- added R11: 100, Resistor_SMD:R_0805_2012Metric_Pad1.20x1.40mm_HandSolder, F.Cu at (182.0, 84.2)
- added R12: 1k, Resistor_SMD:R_0805_2012Metric_Pad1.20x1.40mm_HandSolder, F.Cu at (180.4, 93.8)
- added R2: 10, Resistor_SMD:R_0805_2012Metric_Pad1.20x1.40mm_HandSolder, F.Cu at (144.6, 106.5)
- added R3: 0.1R, Resistor_SMD:R_Shunt_Vishay_WSK2512_6332Metric_T1.19mm, F.Cu at (153.1, 107.1)
- added R4: 4.7k, Resistor_SMD:R_0805_2012Metric_Pad1.20x1.40mm_HandSolder, F.Cu at (112.9, 109.8)
- added R5: 4.7k, Resistor_SMD:R_0805_2012Metric_Pad1.20x1.40mm_HandSolder, F.Cu at (115.2, 109.8)
- added R6: 910k, Resistor_SMD:R_0805_2012Metric_Pad1.20x1.40mm_HandSolder, F.Cu at (163.2, 107.4)
- added R7: 220k, Resistor_SMD:R_0805_2012Metric_Pad1.20x1.40mm_HandSolder, F.Cu at (165.8, 107.4)
- added R8: 10, Resistor_SMD:R_0805_2012Metric_Pad1.20x1.40mm_HandSolder, F.Cu at (121.6, 102.9)
- added R9: 10, Resistor_SMD:R_0805_2012Metric_Pad1.20x1.40mm_HandSolder, F.Cu at (121.6, 106.5)
- added SW1: SW_SPST, Joule Thief-Library:SMD_DPST_Switch, F.Cu at (183.9, 106.5)
- added SW2: SW_SPST, Joule Thief-Library:SMD_DPST_Switch, F.Cu at (103.8, 107.7)
- added U1: INA219AxD, Package_SO:SOIC-8_3.9x4.9mm_P1.27mm, F.Cu at (138.4, 104.8)
- added U2: LTC3105xMS, Package_SO:MSOP-12_3x4.039mm_P0.65mm, F.Cu at (164.3, 102.8)
- added U3: AD5280, Package_SO:TSSOP-14_4.4x5mm_P0.65mm, F.Cu at (176.4, 103.8)
- added U4: INA219AxD, Package_SO:SOIC-8_3.9x4.9mm_P1.27mm, F.Cu at (115.2, 104.8)
- added U5: DW01A, Package_TO_SOT_SMD:SOT-23-6, F.Cu at (182.2, 90.5)
Routing:
- net LITH: track 0.00 -> 142.9 mm
- net V5+: track 0.00 -> 133.4 mm
- net SCL: track 0.00 -> 107.0 mm, vias 0 -> 3
- net SDA: track 0.00 -> 99.1 mm, vias 0 -> 3
- net Net-(BT1--): track 0.00 -> 89.3 mm, vias 0 -> 2
- net Net-(SW1-A): track 0.00 -> 44.7 mm
- net Net-(SW1-B): track 0.00 -> 41.0 mm, vias 0 -> 2
- net Net-(SW2-B): track 0.00 -> 34.7 mm
- net GND: track 0.00 -> 29.9 mm, vias 0 -> 19
- net SHDN: track 0.00 -> 15.8 mm, vias 0 -> 1
- net +ALK: track 0.00 -> 13.2 mm
- net Net-(C9-Pad1): track 0.00 -> 12.6 mm
- net Net-(C2-Pad2): track 0.00 -> 12.4 mm
- net Net-(Q1-D): track 0.00 -> 12.0 mm
- net Net-(U2-SWITCH): track 0.00 -> 10.2 mm
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- added copper zone on B.Cu, net GND
Other:
- board outline added: 88.8 x 55.8 mm
