File: KiCAD/Joule-Thief.kicad_sch (KiCad schematic)
At the start: 30 parts, among them J2 Conn_01x06_Socket, Q4 PMOS, SW1 SW_SPST, SW2 SW_SPST, U2 LTC3105xMS, U3 INA219AxD, U4 LM393, U5 TL431DBZ, U6 DW01A, U7 INA219AxD, U8 AD5280

Commit message: wire up batteries
Parts:
- removed Q4: PMOS, symbol Simulation_SPICE:PMOS
- removed R1: R, symbol Device:R
- removed SW1: SW_SPST, symbol Switch:SW_SPST
- added C5: 0.1u, symbol Device:C_Small
- added C7: C, symbol Device:C_Small
- added J1: AA Cell Clip, symbol Connector_Generic:Conn_01x02
- added J3: Li Cell Clip, symbol Connector_Generic:Conn_01x02
- added Q3, Q5: AO3400A, Package_TO_SOT_SMD:SOT-23, symbol Transistor_FET:AO3400A
- added R10: 100, symbol Device:R
- added R11: 1k, symbol Device:R
- C3: value C -> 4.7u
- L1: value L -> 10u
- R2: value R -> 910k
- R3: value R -> 220k
Connections:
- net +ALK: now also J1.2 (Pin_2)
- net +LITH: now also J3.2 (Pin_2), R10.2
- net MPPC: now also U2.5 (MPPC), U8.1 (A), U8.2 (W); no longer J2.5 (Pin_5)
- net SCL: now also U8.6 (SCL)
- net SDA: now also U8.7 (SDA)
- net VIN: now also R8.4
- net VOUT: now also C7.1
- net VS+: now also U8.13 (VLOG), U8.4 (VDD)
- net at R6.1: no longer D1.2 (A)
- net at R4.1, R5.1, U4.8 (V+): no longer SW2.2 (B)
- net -LITH: now reaches U8.10 (GND)
- net -LITH: now also BTAA.2 (-), C1.2, C2.2, C3.2, C4.2, C6.2, C9.2, J2.2 (Pin_2), R3.2, R7.2, U2.3 (FBLDO), U2.6 (GND), U2.7 (GND), U3.1 (A1), U3.2 (A0), U3.6 (GND), U4.4 (V-), U5.3 (A), U7.1 (A1), U7.6 (GND), U8.11 (VSS), U8.3 (B), U8.8 (AD0), U8.9 (AD1), C7.2, J1.1 (Pin_1), Q3.2 (S), R11.1
- net at U6.1 (OD): now also Q5.1 (G)
- net at U6.2 (CS): now also R11.2
- net at U6.3 (OC): now also Q3.1 (G)
- net at U6.5 (VCC): now also C5.1, R10.1
- net at U6.6 (GND): now also BT18650.2 (-), C5.2, J3.1 (Pin_1), Q5.2 (S)
- net !SHDN: no longer names the net of J2.6 (Pin_6)
- net !SHDN: no longer U2.4 (~{SHDN})
- removed net GND: BT18650.2 (-), BTAA.2 (-), C1.2, C2.2, C3.2, C4.2, C6.2, C9.2, J2.2 (Pin_2), R3.2, R7.2, U2.3 (FBLDO), U2.6 (GND), U2.7 (GND), U3.1 (A1), U3.2 (A0), U3.6 (GND), U4.4 (V-), U5.3 (A), U7.1 (A1), U7.6 (GND)
- new net: Q3.3 (D), Q5.3 (D)
- new net: D1.2 (A), SW2.2 (B)
- new net SHDN: J2.5 (Pin_5), U2.4 (~{SHDN})
- no-connect marks 0 -> 4
Other:
- note removed: "Digital Potentiometer"
- moved on the sheet: BT18650, BTAA, C1, C2, C3, C4, C6, C9, D1, J2, L1, R2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

Commit message: new pcb revision
Parts:
- removed C4: C, symbol Device:C_Small
- removed D1: D_Schottky, symbol Device:D_Schottky
- removed J1: AA Cell Clip, symbol Connector_Generic:Conn_01x02
- removed J3: Li Cell Clip, symbol Connector_Generic:Conn_01x02
- removed R4, R5, R6, R7: R, symbol Device:R
- removed U4: LM393, symbol Comparator:LM393
- removed U5: TL431DBZ, Package_TO_SOT_SMD:SOT-23, symbol Reference_Voltage:TL431DBZ
- added C2, C6, C9: 0.1u, Capacitor_SMD:C_0805_2012Metric_Pad1.18x1.45mm_HandSolder, symbol Device:C_Small
- added R1, R2, R8, R9: 10, Resistor_SMD:R_0805_2012Metric_Pad1.20x1.40mm_HandSolder, symbol Device:R_Small
- added R4, R5: 4.7k, Resistor_SMD:R_0805_2012Metric_Pad1.20x1.40mm_HandSolder, symbol Device:R_Small
- added SW1: SW_SPST, Joule Thief-Library:SMD_DPST_Switch, symbol Switch:SW_SPST
- BATT_1: renamed from BTAA; value Battery_Cell -> Alkaline AA; footprint (none) -> Joule Thief-Library:AA_Cell_Clip
- BT1: renamed from BT18650; footprint (none) -> Joule Thief-Library:18650_Cell_Clip
- C1: renamed from C9; value C_Small -> 0.1u; footprint (none) -> Capacitor_SMD:C_0805_2012Metric_Pad1.18x1.45mm_HandSolder
- C10: renamed from C5; footprint (none) -> Capacitor_SMD:C_0805_2012Metric_Pad1.18x1.45mm_HandSolder
- C3: renamed from C7; value C -> 100u; footprint (none) -> Capacitor_SMD:C_0805_2012Metric_Pad1.18x1.45mm_HandSolder
- C4: renamed from C1; value C -> 10u; footprint (none) -> Capacitor_SMD:C_0805_2012Metric_Pad1.18x1.45mm_HandSolder
- C5: renamed from C2; value C -> 1u; footprint (none) -> Capacitor_SMD:C_0805_2012Metric_Pad1.18x1.45mm_HandSolder
- C7: renamed from C3; footprint (none) -> Capacitor_SMD:C_0805_2012Metric_Pad1.18x1.45mm_HandSolder
- C8: renamed from C6; value C -> 0.1u; footprint (none) -> Capacitor_SMD:C_0805_2012Metric_Pad1.18x1.45mm_HandSolder
- J2: footprint (none) -> Connector_PinSocket_2.54mm:PinSocket_1x06_P2.54mm_Vertical
- L1: footprint (none) -> Joule Thief-Library:Power_Inductor_101040
- R10: renamed from R9; value R_Shunt -> 0.1R; footprint (none) -> Resistor_SMD:R_Shunt_Vishay_WSK2512_6332Metric_T1.19mm
- R11: renamed from R10; footprint (none) -> Resistor_SMD:R_0805_2012Metric_Pad1.20x1.40mm_HandSolder
- R12: renamed from R11; footprint (none) -> Resistor_SMD:R_0805_2012Metric_Pad1.20x1.40mm_HandSolder
- R3: renamed from R8; value R_Shunt -> 0.1R; footprint (none) -> Resistor_SMD:R_Shunt_Vishay_WSK2512_6332Metric_T1.19mm
- R6: renamed from R2; footprint (none) -> Resistor_SMD:R_0805_2012Metric_Pad1.20x1.40mm_HandSolder
- R7: renamed from R3; footprint (none) -> Resistor_SMD:R_0805_2012Metric_Pad1.20x1.40mm_HandSolder
- SW2: footprint (none) -> Joule Thief-Library:SMD_DPST_Switch
- U2: footprint Package_SO:MSOP-12_3x4mm_P0.65mm -> Package_SO:MSOP-12_3x4.039mm_P0.65mm
- renumbered Q3 to Q1, Q5 to Q2, U3 to U1, U8 to U3, U7 to U4, U6 to U5
Connections:
- net +LITH is gone; now on net LITH: BT1.1 (+), R10.4, R11.2
- net VS+ is gone; now on net V5+: J2.1 (Pin_1), U3.13 (VLOG), U3.4 (VDD), U4.2 (A0)
- net SCL: now also R4.2
- net SDA: now also R5.2
- net LITH: now reaches J2.6 (Pin_6)
- net at R3.2: now also C2.1, R1.2; no longer U1.8 (IN+)
- net at R3.3: now also C2.2, R2.2; no longer U1.7 (IN-)
- net at U4.7 (IN-): now also R9.1; no longer R10.3
- net at R10.2: now also C9.2, R8.2; no longer U4.8 (IN+)
- net at R10.1: now also SW2.2 (B)
- net +5V renamed V5+
- net V5+: now also C3.2, R6.1, SW2.1 (A), U2.11 (VOUT), C6.1, R4.1, R5.1
- net -LITH renamed GND
- net GND: now also C3.1, C6.2; no longer C3.2
- net VIN: no longer names the net of C4.1, L1.1, U2.8 (VIN)
- net VIN: now also SW1.1 (A); no longer R3.4
- removed net VOUT: C3.1, R6.1, SW2.1 (A), U2.11 (VOUT)
- new net: C9.1, R10.3, R9.2
- new net: R3.4, SW1.2 (B)
- new net: R8.1, U4.8 (IN+)
- new net: R2.1, U1.7 (IN-)
- new net: R1.1, U1.8 (IN+)
Other:
- note added: "18650 LOAD CELL OC/OCD/SC PROTECT"
- note added: "Address: 0x5E"
- note added: "Changelog: R0V1 -> R0V2 - Add INA219 input filtering - Add SDA/SCL Pullups - Remove Schottky - Rename VS+ to V5+ - Add AD5280 Address"
- note added: "DIGITAL POT 200K MPPC ADJUST"
- note added: "DISC."
- note added: "ENERGY EXTRACTION ALKALINE CELL 1.5V"
- note added: "GPIO TO uC"
- note added: "LOAD CELL POWER MONITOR"
- note added: "LV BOOST CONVERTER 0.250V -> 5.0V"
- note added: "SUPPLY CELL POWER MONITOR"
- note added: "[NEW!]"
- note removed: "18650 cell holder on board or?"
- note removed: "Terminal Blocks to connect to a proper battery holder"
- note removed: "Terminal Blocks to connect to a proper battery pack"
- note removed: "Use PGOOD pin?"
- note removed: "Use the SHDN pin instead"
- note removed: "cell holder on board or? Intention is to be compatible with many alkaline cell sizes"
- moved on the sheet: BATT_1, BT1, C1, C10, C3, C4, C5, C7, C8, J2, L1, Q1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
