File: KiCAD/Joule-Thief_R2.kicad_pcb (KiCad board)
At the start: 2 copper layers, 90.1 x 58.2 mm, 35 parts, among them J2 Conn_01x06_Socket, Q1 AO3400A, Q2 AO3400A, SW1 SW_SPST, SW2 SW_SPST, U1 INA219AxD, U2 LTC3105xMS, U3 AD5280, U4 INA219AxD, U5 DW01A

Commit message: made pcb r3, start r4
Parts:
- moved C4 49.3 mm to (163.4, 99.1)
- moved C3 49.0 mm to (157.6, 104.2)
- moved BATT_1 48.8 mm to (130.8, 92.7)
- moved BT1 48.8 mm to (140.3, 71.6)
- moved C10 48.8 mm to (182.0, 86.6)
- moved C7 48.8 mm to (168.7, 104.8)
- moved Q2 48.8 mm to (177.1, 90.5)
- moved R1 48.8 mm to (144.7, 102.9)
- moved R10 48.8 mm to (130.6, 107.3)
- moved R11 48.8 mm to (182.0, 84.2)
- moved R12 48.8 mm to (180.4, 93.8)
- moved R2 48.8 mm to (144.6, 106.5)
- moved R4 48.8 mm to (112.9, 109.8)
- moved U2 48.8 mm to (164.3, 102.8)
- moved U3 48.8 mm to (176.4, 103.8)
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Routing:
- net LITH: track 111.5 -> 142.9 mm, vias 1 -> 0
- net V5+: track 136.0 -> 133.4 mm
- net Net-(SW1-B): track 43.5 -> 41.0 mm
- net SCL: track 105.3 -> 107.0 mm
- net SDA: track 100.4 -> 99.1 mm
- net Net-(Q1-D): track 11.0 -> 12.0 mm
- net GND: track 30.5 -> 29.9 mm, vias 17 -> 19
- net Net-(BT1--): track 89.7 -> 89.3 mm, vias 0 -> 2
Other:
- board size 90.1 x 58.2 mm -> 88.8 x 55.8 mm
