File: KiCAD/Joule-Thief_R3.kicad_pcb (KiCad board)
At the start: 2 copper layers, 90.1 x 58.2 mm, 35 parts, among them J2 Conn_01x06_Socket, Q1 AO3400A, Q2 AO3400A, SW1 SW_SPST, SW2 SW_SPST, U1 INA219AxD, U2 LTC3105xMS, U3 AD5280, U4 INA219AxD, U5 DW01A

Commit message: made pcb r3, start r4
Changed lines of the file:
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@@
 		(at 101.2475 42.405)
 		(property "Reference" "BT1"
-			(at 36.4025 -2.955 270)
+			(at 0 0 0)
 			(unlocked yes)
 			(layer "F.SilkS")
@@
 				(font
 					(size 1 1)
-					(thickness 0.1)
+					(thickness 0.16)
 				)
 			)
@@
 		(pad "1" thru_hole circle
 			(at 36.45 0)
-			(size 2 2)
+			(size 2.5 2.5)
 			(drill 1.2)
 			(layers "*.Cu" "*.Mask")
@@
 		(pad "2" thru_hole circle
 			(at -36.45 0)
-			(size 2 2)
+			(size 2.5 2.5)
 			(drill 1.2)
 			(layers "*.Cu" "*.Mask")
@@
 		(at 91.7475 63.505)
 		(property "Reference" "BATT_1"
-			(at 27.4025 -3.705 270)
+			(at 0 0 0)
 			(unlocked yes)
 			(layer "F.SilkS")
@@
 				(font
 					(size 1 1)
-					(thickness 0.1)
+					(thickness 0.16)
 				)
 			)
@@
 				(font
 					(size 1 1)
-					(thickness 0.15)
+					(thickness 0.16)
 				)
 			)
@@
 				(font
 					(size 1 1)
-					(thickness 0.15)
+					(thickness 0.16)
 				)
 			)
@@
 				(font
 					(size 1 1)
-					(thickness 0.15)
+					(thickness 0.16)
 				)
 			)
@@
 				(font
 					(size 1 1)
-					(thickness 0.15)
+					(thickness 0.16)
 				)
 			)
@@
 				(font
 					(size 1 1)
-					(thickness 0.15)
+					(thickness 0.16)
 				)
 			)
@@
 				(font
 					(size 1 1)
-					(thickness 0.15)
+					(thickness 0.16)
 				)
 			)
@@
 				(font
 					(size 1 1)
-					(thickness 0.15)
+					(thickness 0.16)
 				)
 			)
@@
 				(font
 					(size 1 1)
-					(thickness 0.15)
+					(thickness 0.16)
 				)
 			)
@@
 				(font
 					(size 1 1)
-					(thickness 0.15)
+					(thickness 0.16)
 				)
 			)
@@
 				(font
 					(size 1 1)
-					(thickness 0.15)
+					(thickness 0.16)
 				)
 			)
@@
 				(font
 					(size 1 1)
-					(thickness 0.15)
+					(thickness 0.16)
 				)
 			)
@@
 				(font
 					(size 1 1)
-					(thickness 0.15)
+					(thickness 0.16)
 				)
 			)
@@
 				(font
 					(size 1 1)
-					(thickness 0.15)
+					(thickness 0.16)
 				)
 			)
@@
 				(font
 					(size 1 1)
-					(thickness 0.15)
+					(thickness 0.16)
 				)
 			)
@@
 				(font
 					(size 1 1)
-					(thickness 0.15)
+					(thickness 0.16)
 				)
 			)
@@
 				(font
 					(size 1 1)
-					(thickness 0.15)
+					(thickness 0.16)
 				)
 			)
@@
 				(font
 					(size 1 1)
-					(thickness 0.15)
+					(thickness 0.16)
 				)
 			)
@@
 				(font
 					(size 1 1)
-					(thickness 0.15)
+					(thickness 0.16)
 				)
 			)
@@
 				(font
 					(size 1 1)
-					(thickness 0.15)
+					(thickness 0.16)
 				)
 			)
@@
 				(font
 					(size 1 1)
-					(thickness 0.15)
+					(thickness 0.16)
 				)
 			)
@@
 				(font
 					(size 1 1)
-					(thickness 0.15)
+					(thickness 0.16)
 				)
 			)
@@
 				(font
 					(size 1 1)
-					(thickness 0.15)
+					(thickness 0.16)
 				)
 			)
@@
 		(tags "SMD Power Inductor")
 		(property "Reference" "L1"
-			(at 0 7 270)
+			(at 0 0 0)
 			(unlocked yes)
 			(layer "F.SilkS")
@@
 				(font
 					(size 1 1)
-					(thickness 0.1)
+					(thickness 0.16)
 				)
 			)
@@
 				(font
 					(size 1 1)
-					(thickness 0.15)
+					(thickness 0.16)
 				)
 			)
@@
 				(font
 					(size 1 1)
-					(thickness 0.15)
+					(thickness 0.16)
 				)
 			)
@@
 				(font
 					(size 1 1)
-					(thickness 0.15)
+					(thickness 0.16)
 				)
 			)
@@
 		(tags "SMD_DPST_Switch")
 		(property "Reference" "SW1"
-			(at -6.15 -1.7 0)
+			(at 6.45 -1.65 0)
 			(unlocked yes)
 			(layer "F.SilkS")
@@
 				(font
 					(size 1 1)
-					(thickness 0.1)
+					(thickness 0.16)
 				)
 			)
@@
 				(font
 					(size 1 1)
-					(thickness 0.15)
+					(thickness 0.16)
 				)
 			)
@@
 				(font
 					(size 1 1)
-					(thickness 0.15)
+					(thickness 0.16)
 				)
 			)
@@
 				(font
 					(size 1 1)
-					(thickness 0.15)
+					(thickness 0.16)
 				)
 			)
@@
 				(font
 					(size 1 1)
-					(thickness 0.15)
+					(thickness 0.16)
 				)
 			)
@@
 				(font
 					(size 1 1)
-					(thickness 0.15)
+					(thickness 0.16)
 				)
 			)
@@
 		(tags "SMD_DPST_Switch")
 		(property "Reference" "SW2"
-			(at -6.3 1.65 0)
+			(at -6.45 -1.6 0)
 			(unlocked yes)
 			(layer "F.SilkS")
@@
 				(font
 					(size 1 1)
-					(thickness 0.1)
+					(thickness 0.16)
 				)
 			)
