File: KiCAD/Joule-Thief_R4.kicad_pcb (KiCad board)
At the start: 2 copper layers, 90.1 x 58.2 mm, 35 parts, among them J2 Conn_01x06_Socket, Q1 AO3400A, Q2 AO3400A, SW1 SW_SPST, SW2 SW_SPST, U1 INA219AxD, U2 LTC3105xMS, U3 AD5280, U4 INA219AxD, U5 DW01A

Commit message: made pcb r3, start r4
Parts:
- moved BT1 3.13 mm to (104.4, 42.3)
- moved Q1 3.13 mm to (146.3, 67.7)
- moved Q2 3.13 mm to (141.1, 61.3)
- moved R11 3.13 mm to (146.1, 54.9)
- moved C10 3.13 mm to (146.1, 57.3)
- moved R12 3.13 mm to (144.5, 64.5)
- moved U5 3.13 mm to (146.3, 61.3)
- moved L1 1.07 mm to (129.2, 60.5), turned to 0 degrees
Routing:
- net Net-(SW1-A): track 45.0 -> 5.41 mm
- net Net-(BT1--): track 89.7 -> 92.8 mm
- net Net-(U2-SWITCH): track 10.2 -> 7.21 mm
- net LITH: track 111.5 -> 109.7 mm
- net Net-(Q1-D): track 11.0 -> 12.2 mm
- added copper zone on F.Cu, net Net-(SW1-A)
- added copper zone on F.Cu, net Net-(U2-SWITCH)
