File: KiCAD/Joule-Thief_R5.kicad_pcb (KiCad board)
At the start: 2 copper layers, 90.9 x 59.5 mm, 35 parts, among them J2 Conn_01x06_Socket, Q1 AO3400A, Q2 AO3400A, SW1 SW_SPST, SW2 SW_SPST, U1 INA219AxD, U2 LTC3105xMS, U3 AD5280, U4 INA219AxD, U5 DW01A

Commit message: r5 is the one bro i swear
Routing:
- net V5+: track 124.5 -> 130.7 mm
- net GND: track 51.9 -> 49.0 mm, vias 14 -> 15
- net SCL: track 107.5 -> 106.7 mm
Other:
- board text added: "><>*"
- board text added: "JOULE THIEF R0"
