File: KiCAD/Joule Thief R1/Joule_Thief_R1.kicad_sch (KiCad schematic)
At the start: 110 parts, among them J1 Conn_01x06, J3 Conn_01x06, J4 Conn_01x06, J5 Conn_01x06, J6 Conn_01x06, J7 Conn_01x06, J8 Conn_01x06, J9 Conn_01x06, Q1 AO3400A, Q2 AO3400A, Q3 AO3400A, SW1 SW_DPDT_x2, U11 INA219AxD, U12 INA219AxD, U13 INA219AxD, U2 LTC3105xMS, U3 AD5280, U5 DW01A, U7 LTC3105xMS, U8 AD5280, U9 INA219AxD

Commit message: both schematics finished
Parts:
- removed C13: 10u, Capacitor_SMD:C_0805_2012Metric_Pad1.18x1.45mm_HandSolder, symbol Device:C_Small
- removed C14: 1u, Capacitor_SMD:C_0805_2012Metric_Pad1.18x1.45mm_HandSolder, symbol Device:C_Small
- removed C15, C18, C19, C21, C23: 0.1u, Capacitor_SMD:C_0805_2012Metric_Pad1.18x1.45mm_HandSolder, symbol Device:C_Small
- removed C16: 4.7u, Capacitor_SMD:C_0805_2012Metric_Pad1.18x1.45mm_HandSolder, symbol Device:C_Small
- removed C17: 100u, symbol Device:C_Small
- removed C20, C22: 1F, symbol Device:C_Polarized_US
- removed J3, J4, J5, J6, J7, J8, J9: Conn_01x06, symbol Connector_Generic:Conn_01x06
- removed JP29, JP30, JP31, JP32, JP33, JP34, JP35, JP36, JP37, JP38, JP39, JP40, JP41, JP42, JP43, JP44, JP45, JP46, JP47, JP48: SolderJumper_2_Open, symbol Jumper:SolderJumper_2_Open
- removed L2: 10u, Joule Thief-Library:Power_Inductor_101040, symbol Device:L
- removed LITH2: 18650, Joule Thief-Library:18650_Cell_Clip, symbol Device:Battery_Cell
- removed Q1, Q2, Q3: AO3400A, Package_TO_SOT_SMD:SOT-23, symbol Transistor_FET:AO3400A
- removed R11: 100, Resistor_SMD:R_0805_2012Metric_Pad1.20x1.40mm_HandSolder, symbol Device:R
- removed R12: 1k, Resistor_SMD:R_0805_2012Metric_Pad1.20x1.40mm_HandSolder, symbol Device:R
- removed R14: 1M, Resistor_SMD:R_0805_2012Metric_Pad1.20x1.40mm_HandSolder, symbol Device:R
- removed R15: 220k, Resistor_SMD:R_0805_2012Metric_Pad1.20x1.40mm_HandSolder, symbol Device:R
- removed R16, R18, R20, R22: 10, Resistor_SMD:R_0805_2012Metric_Pad1.20x1.40mm_HandSolder, symbol Device:R_Small
- removed R17, R21: 0.1R, Resistor_SMD:R_Shunt_Vishay_WSK2512_6332Metric_T1.19mm, symbol Device:R_Shunt
- removed R19: 10k, Resistor_SMD:R_0805_2012Metric_Pad1.20x1.40mm_HandSolder, symbol Device:R_Small
- removed TPx1: TestPoint_Alt, symbol Connector:TestPoint_Alt
- removed U10: ~, symbol Joule_Thief_R1:BMS_BOARD
- removed U11, U9: INA219AxD, Package_SO:SOIC-8_3.9x4.9mm_P1.27mm, symbol Sensor_Energy:INA219AxD
- removed U5: DW01A, Package_TO_SOT_SMD:SOT-23-6, symbol Battery_Management:DW01A
- removed U7: LTC3105xMS, Package_SO:MSOP-12_3x4.039mm_P0.65mm, symbol Regulator_Switching:LTC3105xMS
- removed U8: AD5280, Package_SO:TSSOP-14_4.4x5mm_P0.65mm, symbol Potentiometer_Digital:AD5280
- added R10: 1k, Resistor_SMD:R_0805_2012Metric_Pad1.20x1.40mm_HandSolder, symbol Device:R_Small
- added R9: 100, Resistor_SMD:R_0805_2012Metric_Pad1.20x1.40mm_HandSolder, symbol Device:R_Small
- added U5: DW01, Package_TO_SOT_SMD:SOT-23-6_Handsoldering, symbol 000_Dropbin:DW01
- added U6: FS8205A, Package_TO_SOT_SMD:SOT-23-6_Handsoldering, symbol 000_Dropbin:FS8205A
- renumbered C24 to C1, C25 to C2, C7 to C6, C6 to C7, C26 to C8, C27 to C9, JP49 to JP1, JP14 to JP10, JP57 to JP13, JP58 to JP14, JP59 to JP15, JP60 to JP16, JP61 to JP17, JP62 to JP18, JP63 to JP19, JP50 to JP2, JP64 to JP20, JP51 to JP3, JP52 to JP4, JP53 to JP5, JP54 to JP6, JP55 to JP7, JP56 to JP8, JP13 to JP9, R24 to R1, R23 to R2, R25 to R3, R6 to R4, R7 to R5, R27 to R6, R26 to R7, R28 to R8, TPx to TPx1, U12 to U1, U13 to U4
Connections:
- net GND: now also R10.1, U6.6 (S2), U6.7 (S2)
- net at C10.2: now also SW1.4 (A), R9.1, U5.5 (VCC); no longer LITH1.2 (-)
- net BAT+: now reaches LITH1.1 (+)
- net BAT+: now also R9.2; no longer SW1.4 (A)
- net BAT-: now reaches C10.1
- net BAT-: now also LITH1.2 (-), U5.6 (GND), U6.2 (S1), U6.3 (S1)
- new net: U5.1 (OD), U6.4 (G1)
- new net: R10.2, U5.2 (CS)
- new net: U5.3 (OC), U6.5 (G2)
- no-connect marks 8 -> 7
Other:
- note added: "18650 BMS MODULE"
- note removed: "18650 LOAD CELL OC/OCD/SC PROTECT"
- note removed: "1F SUPERCAP"
- note removed: "Changelog: R0V1 -> R0V2 - Add INA219 input filtering - Add SDA/SCL Pullups - Remove Schottky - Rename VS+ to V5+ - Add AD5280 Address"
- note removed: "GENERIC BMS MODULE"
- note removed: "MAIN BOARD"
- note removed: "MODULE 1"
- note removed: "MODULE 2"
- note removed: "MODULE 3"
- note removed: "MODULE 4"
- note removed: "MODULE 5"
- note removed: "MODULE 6"
- note removed: "MODULE 7"
- note removed: "[NEW!]"
- moved on the sheet: BATT_1, C1, C2, C3, C4, C5, C6, C7, C8, C9, D1, J1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

Commit message: layout extraction module
Parts:
- removed TPx1: TestPoint_Alt, symbol Connector:TestPoint_Alt
- BATT_1: footprint Joule Thief-Library:AA_Cell_Clip -> 000_Dropbin:AA_Cell_Clip_V2
- C3: footprint (none) -> Capacitor_THT:CP_Radial_D5.0mm_P2.00mm
- D1: footprint (none) -> Diode_THT:D_DO-41_SOD81_P10.16mm_Horizontal
- J1: footprint (none) -> Connector_JST:JST_PH_B6B-PH-K_1x06_P2.00mm_Vertical
- JP1, JP10, JP11, JP12, JP13, JP14, JP15, JP16, JP17, JP18, JP19, JP2, JP20, JP3, JP4, JP5, JP6, JP7, JP8, JP9: footprint (none) -> Jumper:SolderJumper-2_P1.3mm_Open_RoundedPad1.0x1.5mm
- L1: footprint Joule Thief-Library:Power_Inductor_101040 -> 000_Dropbin:Power_Inductor_101040
- LITH1: footprint Joule Thief-Library:18650_Cell_Clip -> 000_Dropbin:18650_Cell_Clip_V2
- R1, R6: footprint Resistor_SMD:R_Shunt_Vishay_WSK2512_6332Metric_T1.19mm -> 000_Dropbin:R_Shunt_2512_V2
- SW1: footprint (none) -> 000_Dropbin:SS22F25_DPDT_Straight_V2
- U7: renamed from U6; footprint Package_TO_SOT_SMD:SOT-23-6_Handsoldering -> Package_TO_SOT_SMD:SOT-23-8_Handsoldering
Connections:
- net GND: now also J1.5 (Pin_5); no longer J1.2 (Pin_2)
- net SHDN: now also J1.1 (Pin_1); no longer J1.5 (Pin_5)
- net VBOOST: now also SW1.2 (B); no longer SW1.1 (A)
- net VBUS: now also SW1.4 (A); no longer SW1.2 (B)
- net VCC: now also J1.6 (Pin_6), SW1.6 (C); no longer J1.1 (Pin_1), SW1.3 (C)
- net VOUT: now also J1.2 (Pin_2); no longer J1.6 (Pin_6)
- net at C10.2, R9.1, U5.5 (VCC): now also SW1.1 (A); no longer SW1.4 (A)
- net at D1.2 (A): now also SW1.3 (C); no longer SW1.6 (C)
- no-connect marks 7 -> 8
Other:
- moved on the sheet: D1, SW1A, SW1B
